File: KiCAD/load_pull/load_pull.kicad_pcb (KiCad board)
At the start: 2 copper layers, 28 parts, among them J1 Conn_Coaxial, J2 Conn_Coaxial, U1 TLV3542IDR, U2 LT1206CR-PBF

Commit message: Up plane
Routing:
- net -12V: track 75.4 -> 105.1 mm
- added copper zone on F.Cu, net GND
Changed lines of the file:
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@@
+	)
+	(segment
+		(start 118.618 81.407)
+		(end 119.706 82.495)
+		(width 1.2)
+		(layer "F.Cu")
+		(net 1)
 	)
 	(segment
@@
 	)
 	(segment
+		(start 131.191 63.754)
+		(end 123.698 71.247)
+		(width 1.2)
+		(layer "F.Cu")
+		(net 1)
+	)
+	(segment
 		(start 128.325 83.892)
 		(end 128.198 83.765)
@@
 	)
 	(segment
+		(start 123.698 71.247)
+		(end 119.761 71.247)
+		(width 1.2)
+		(layer "F.Cu")
+		(net 1)
+	)
+	(segment
 		(start 126.674 83.765)
 		(end 125.404 82.495)
@@
 	)
 	(segment
+		(start 119.706 82.495)
+		(end 121.086 82.495)
+		(width 1.2)
+		(layer "F.Cu")
+		(net 1)
+	)
+	(segment
+		(start 131.191 62.103)
+		(end 131.191 63.754)
+		(width 1.2)
+		(layer "F.Cu")
+		(net 1)
+	)
+	(segment
 		(start 147.955 82.5246)
 		(end 147.955 80.772)
@@
 	)
 	(segment
+		(start 119.761 71.247)
+		(end 118.618 72.39)
+		(width 1.2)
+		(layer "F.Cu")
+		(net 1)
+	)
+	(segment
 		(start 131.191 60.325)
 		(end 132.461 59.055)
@@
 	)
 	(segment
+		(start 118.618 72.39)
+		(end 118.618 81.407)
+		(width 1.2)
+		(layer "F.Cu")
+		(net 1)
+	)
+	(segment
 		(start 128.198 83.765)
 		(end 126.674 83.765)
@@
 	)
 	(segment
+		(start 134.493 76.852)
+		(end 134.493 76.581)
+		(width 0.3)
+		(layer "F.Cu")
+		(net 3)
+	)
+	(segment
 		(start 134.493 76.581)
 		(end 137.287 73.787)
@@
 		(start 147.701 71.628)
 		(end 145.415 73.914)
+		(width 0.3)
+		(layer "F.Cu")
+		(net 3)
+	)
+	(segment
+		(start 134.548 76.907)
+		(end 134.493 76.852)
 		(width 0.3)
 		(layer "F.Cu")
@@
 		(layer "F.Cu")
 		(net 13)
+	)
+	(zone
+		(net 2)
+		(net_name "GND")
+		(layer "F.Cu")
+		(name "g_plane")
+		(hatch none 0.5)
+		(connect_pads
+			(clearance 0.5)
+		)
+		(min_thickness 0.25)
+		(filled_areas_thickness no)
+		(fill yes
+			(thermal_gap 0.5)
+			(thermal_bridge_width 0.5)
+			(island_removal_mode 1)
+			(island_area_min 10)
+		)
+		(polygon
+			(pts
+				(xy 99.06 100.076) (xy 100.711 101.727) (xy 173.101 101.727) (xy 174.752 100.076) (xy 174.752 61.468)
+				(xy 170.815 57.531) (xy 99.06 57.531)
+			)
+		)
 	)
 	(zone
@@
 		(name "groun_plane")
 		(hatch none 0.5)
+		(priority 1)
 		(connect_pads
 			(clearance 0.5)

Commit message: Docs start of project
Parts:
- added G***: LOGO, Logo:SEA_logo_small, F.Cu at (111.5, 70.4)
Routing:
- net Net-(U2-+IN): track 4.80 -> 4.16 mm
- net GND: vias 19 -> 320
Other:
- board outline added: 76.5 x 46 mm
- board text added: "LF - Load Pull"
