File: KiCAD/RF_driver/RF_driver/RF_driver.kicad_sch (KiCad schematic)
At the start: 17 parts, among them J1 Conn_Coaxial, J2 Conn_01x02_Pin, U1 TLV3542IDR

Commit message: Changes
Parts:
- Rf2: value 10k -> 0
Changed lines of the file:
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@@
 			)
 		)
-		(property "Value" "10k"
+		(property "Value" "0"
 			(at 125.73 104.14 90)
 			(effects

Commit message: Design ordered
Parts:
- removed C2: 10nF, Capacitor_SMD:C_0805_2012Metric_Pad1.18x1.45mm_HandSolder, symbol Device:C
- removed C3: 1nF, Capacitor_SMD:C_0805_2012Metric_Pad1.18x1.45mm_HandSolder, symbol Device:C
- removed Rf1, Rg1: 10k, Resistor_SMD:R_0805_2012Metric_Pad1.20x1.40mm_HandSolder, symbol Device:R
- removed U1: TLV3542IDR, D8_TEX, symbol HF_opamp:TLV3542IDR
- added U1: TLV3541IDBVR, RF_PA:DBV0005A_N, symbol HF_opamp:TLV3541IDBVR
- C1, C4: LCSC (none) -> C49678
- C5: LCSC (none) -> C1710
- C6: LCSC (none) -> C46653
- C7: value 1nF -> 100nF; LCSC (none) -> C49678
- Rf2: LCSC (none) -> C17477
- Rg2: LCSC (none) -> C17414
- Rz1, Rz2: LCSC (none) -> C17408
Connections:
- net GND: now also Con1.2 (pin2), U1.2 (V-); no longer C1.2, Rz1.1
- net at C7.2, Rf2.2: now also U1.1 (OUT)
- net at Rf2.1, Rg2.2: now also U1.4 (IN-)
- net +12V renamed +5V
- net +5V: now also Rz1.2, U1.5 (V+)
- net -12V: no longer names the net of C1.1
- net -12V: now also Rz1.1, Rz2.2, U1.3 (IN+); no longer Con1.2 (pin2)
- new net: C1.2, J1.1 (In)
Other:
- moved on the sheet: Rz1
